File: ComAir.kicad_pcb (KiCad board)
At the start: 2 copper layers, 90.5 x 28 mm, 69 parts, among them J101 Conn_01x02, J102 Conn_01x02, J103 Conn_01x05, J104 Conn_01x07, J105 Conn_01x07, J401 DX07S016JA1R1500, SW101 SW_Push, SW102 SW_Push, U101 STM32L431CBUx, U102 12BHC186P1-GR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

Commit message: PCB ready for first prototype production
Signed-off-by: Alexis Jeandet <alexis.jeandet@member.fsf.org>
Other:
- board text added: "CC-BY-SA"
- board text added: "ComAir V1.0 LPP/CNRS"
